Commit message: pick and place procedure complete

File: p26_robot/p26_robot/urdf/p26_lefty.urdf (robot description, URDF)
Before this commit: robot p26_lefty, 26 links, 25 joints
Links:
- link lefty_tool: geometry collision mesh filename=package://p26_robot/meshes/tool0/collision/manipulator_coll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; visual mesh filename=package://p26_robot/meshes/tool0/visual/manipulator.STL

File: p26_robot/p26_robot/urdf/p26_lefty.xacro (robot description, xacro)
@@ -16,14 +16,15 @@
   <link name="${prefix}tool">
     <visual>
-    <origin xyz="0.03 -0.0625 -0.1" rpy="0 -1.57079632 0"/>
+    <origin xyz="0 0 0" rpy="0.785398 0 0"/>
       <geometry>
-        <mesh filename="package://p26_robot/meshes/tool0/visual/tool0.STL" scale="0.001 0.001 0.001" />
+        <mesh filename="package://p26_robot/meshes/tool0/visual/manipulator.STL"/>
       </geometry>
       <xacro:material_abb_white />
     </visual>
     <collision>
-    <origin xyz="0.03 -0.0625 -0.1" rpy="0 -1.57079632 0"/>
+<!--    <origin xyz="0 0 0" rpy="1.5707963 -2.3561943 1.5707963"/>-->
+    <origin xyz="0 0 0" rpy="0.785398 0 0"/><!--0.785398 -1.5707963 3.14159265"/> 2.3561943-->
       <geometry>
-        <mesh filename="package://p26_robot/meshes/tool0/collision/tool0.STL" scale="0.001 0.001 0.001" />
+        <mesh filename="package://p26_robot/meshes/tool0/collision/manipulator_collision.STL"/>
       </geometry>
       <xacro:material_abb_white />
